Commit message: Update ur_common.xacro

File: ur_description/urdf/inc/ur_common.xacro (robot description, xacro)
@@ -27,5 +27,5 @@
     <xacro:get_visual_params />
     <xacro:if value="${force_abs_paths}">
-      <xacro:property name="mesh" value="file://$(find ${visual_params['mesh']['package']})/${visual_params['mesh']['path']}" scope="parent"/>
+      <xacro:property name="mesh" value="$(find ${visual_params['mesh']['package']})/${visual_params['mesh']['path']}" scope="parent"/>
     </xacro:if>
     <xacro:unless value="${force_abs_paths}">
