Commit message: us probe stl models

File: c5_2_60_description/urdf/c5_2_60.xacro (robot description, xacro)
@@ -1,5 +1,54 @@
 <?xml version="1.0" ?>
-<robot xmlns:xacro="http://www.ros.org/wiki/xacro" name="probe">
+<robot xmlns:xacro="http://www.ros.org/wiki/xacro" xmlns:ignition="http://gazebosim.org/schema" name="probe">
   <xacro:macro name="c5_2_60" params="parent name *origin">
+    <material name="white">
+      <color rgba="1 1 1 1"/>
+    </material>
+    <link name="${name}_link">
+      <collision>
+	<geometry>
+          <mesh filename="file://$(find c5_2_60_description)/meshes/c5_2_60.stl"/>
+	</geometry>
+      </collision>
+      <visual>
+	<geometry>
+          <mesh filename="file://$(find c5_2_60_description)/meshes/c5_2_60.stl"/>
+	</geometry>
+	<material  name="white"/>
+      </visual>
+      <inertial>
+	<origin xyz="0 0 0" rpy="0 0 0"/>
+	<mass value="0.030"/>
+	<inertia ixx="1.75e-5" ixy="0" ixz="0" iyy="1.75e-5" iyz="0" izz="1.75e-5"/>
+      </inertial>
+    </link>
+    <!-- Define the probe sensor -->
+    <gazebo reference="${name}_link">
+      <sensor name="us" type="custom" ignition:type="USSensor">
+	<always_on>1</always_on>
+	<topic> image_us </topic>
+	<US>
+	  <!-- These are specific to PlusTK -->
+	  <PlusDir> $(find ignition_gazebo_us_system)/config</PlusDir>
+	  <PlusConfig> config-ismr.xml </PlusConfig>
+	</US>
+      </sensor>
+    </gazebo>
+    <joint name="${name}_joint" type="fixed">
+      <parent link="${parent}"/>
+      <child link="${name}_link"/>
+      <origin xyz="0 -0.05 0.10" rpy="0 0 1.5708"/>
+    </joint>
+    <gazebo reference="${name}_joint">
+      <preserveFixedJoint>true</preserveFixedJoint>
+      <sensor type="force_torque" name="ft_sensor">
+	<always_on>true</always_on>
+	<pose>0 0 0 0 0 0</pose>
+	<visualize>true</visualize>
+	<update_rate>50</update_rate>
+	<topic>ft_probe</topic>
+	<ignition_frame_id>${name}_link</ignition_frame_id>
+      </sensor>
+    </gazebo>
   </xacro:macro>
 </robot>

Commit message: Update c5_2_60.xacro

File: c5_2_60_description/urdf/c5_2_60.xacro (robot description, xacro)
@@ -8,10 +8,10 @@
       <collision>
 	<geometry>
-          <mesh filename="file://$(find c5_2_60_description)/meshes/c5_2_60.stl"/>
+          <mesh filename="$(find c5_2_60_description)/meshes/c5_2_60.stl"/>
 	</geometry>
       </collision>
       <visual>
 	<geometry>
-          <mesh filename="file://$(find c5_2_60_description)/meshes/c5_2_60.stl"/>
+          <mesh filename="$(find c5_2_60_description)/meshes/c5_2_60.stl"/>
 	</geometry>
 	<material  name="white"/>

Commit message: standalone pluslib and small fixes to US frames

File: c5_2_60_description/urdf/c5_2_60.xacro (robot description, xacro)
@@ -8,10 +8,10 @@
       <collision>
 	<geometry>
-          <mesh filename="$(find c5_2_60_description)/meshes/c5_2_60.stl"/>
+          <mesh filename="$(find c5_2_60_description)/meshes/c5_2_60.dae"/>
 	</geometry>
       </collision>
       <visual>
 	<geometry>
-          <mesh filename="$(find c5_2_60_description)/meshes/c5_2_60.stl"/>
+          <mesh filename="$(find c5_2_60_description)/meshes/c5_2_60.dae"/>
 	</geometry>
 	<material  name="white"/>
@@ -38,5 +38,5 @@
       <parent link="${parent}"/>
       <child link="${name}_link"/>
-      <origin xyz="0 -0.05 0.10" rpy="0 0 1.5708"/>
+      <origin xyz="0 -0.05 0.10" rpy="1.5708 0 -1.5708"/>
     </joint>
     <gazebo reference="${name}_joint">
